Commit message: "Managed to get odom to show up once controller_manager was removed"

File: articubot_one/description/camera.xacro (robot description, xacro)
@@ -32,5 +32,5 @@
             <pose> 0 0 0 0 0 0 </pose>
             <visualize>true</visualize>
-            <update_rate>10</update_rate>
+            <update_rate>1</update_rate>
             <camera>
                 <horizontal_fov>1.089</horizontal_fov>

File: articubot_one/description/gazebo_control.xacro (robot description, xacro)
@@ -8,5 +8,5 @@
             <!-- kinematics -->
             <wheel_separation>0.35</wheel_separation>
-            <wheel_radius>0.5</wheel_radius>
+            <wheel_diameter>1.0</wheel_diameter>
             <topic>cmd_vel</topic>
             <!-- limits -->
@@ -33,16 +33,5 @@
             <frame_id>odom</frame_id>
             <child_frame_id>base_footprint</child_frame_id>
-            <odom_publish_frequency>20</odom_publish_frequency>
-        </plugin>
-    </gazebo>
-    <gazebo>
-        <plugin filename="ignition-gazebo-odometry-publisher-system" name="ignition::gazebo::systems::OdometryPublisher">
-            <odom_frame> map</odom_frame>
-            <robot_base_frame> base_footprint</robot_base_frame>
-            <odom_publish_frequency>20.0</odom_publish_frequency>
-            <odom_topic>odom</odom_topic>
-            <tf_topic>tf</tf_topic>
-            <gaussian_noise>5.0</gaussian_noise>
-            <xyz_offset>0 0 0</xyz_offset>
+            <odom_publish_frequency>50</odom_publish_frequency>
         </plugin>
     </gazebo>

File: articubot_one/description/lidar.xacro (robot description, xacro)
@@ -30,13 +30,14 @@
     </link>
     <gazebo reference="laser_frame">
-        <material>Gazebo/Black</material>
-        <sensor name="laser" type="ray">
-            <pose> 0 0 0 0 0 0 </pose>
-            <visualize>false</visualize>
-            <update_rate>10</update_rate>
+           <material>Gazebo/FlatBlack</material>
+        <sensor type="ray" name="laser">
+            <pose>0 0 0 0 0 0</pose>
+            <visualize>true</visualize>
+            <update_rate>1</update_rate>
             <ray>
                 <scan>
                     <horizontal>
                         <samples>360</samples>
+                        <resolution>1</resolution>
                         <min_angle>-3.14</min_angle>
                         <max_angle>3.14</max_angle>
@@ -46,4 +47,5 @@
                     <min>0.3</min>
                     <max>12</max>
+                    <resolution>0.01</resolution>
                 </range>
             </ray>
@@ -51,4 +53,5 @@
                 <ros>
                     <argument>~/out:=scan</argument>
+                    <!-- <argument>ros-args -r ~/out:=scan</argument> -->
                 </ros>
                 <output_type>sensor_msgs/LaserScan</output_type>

File: articubot_one/description/robot.urdf.xacro (robot description, xacro)
@@ -1,16 +1,8 @@
 <?xml version="1.0"?>
-<robot xmlns:xacro="http://www.ros.org/wiki/xacro"  name="robot">
-    <xacro:arg name="use_ros2_control" default="false"/>
-    <xacro:arg name="sim_mode" default="false"/>
-    <xacro:include filename="robot_core.xacro" />
-    <xacro:if value="$(arg use_ros2_control)">
-        <xacro:include filename="ros2_control.xacro" />
-    </xacro:if>
-    <xacro:unless value="$(arg use_ros2_control)">
-        <xacro:include filename="gazebo_control.xacro" />
-    </xacro:unless>
-    <xacro:include filename="lidar.xacro" />
+<robot xmlns:xacro="http://www.ros.org/wiki/xacro" name="articubot">
+    <xacro:include filename="robot_core.xacro"/>
+    <xacro:include filename="lidar.xacro"/>
+    <xacro:include filename="face.xacro" />
     <xacro:include filename="camera.xacro" />
-    <!-- <xacro:include filename="depth_camera.xacro" /> -->
-    <xacro:include filename="face.xacro" />
+    <xacro:include filename="gazebo_control.xacro"/>
 </robot>
