Commit message: "Fixed transforms to correct standardised form"

File: src/articubot_one/description/gazebo_control.xacro (robot description, xacro)
@@ -3,35 +3,18 @@
     <gazebo>
         <plugin name="diff_drive" filename="libgazebo_ros_diff_drive.so">
-             <!-- wheels -->
+            <!-- Wheel Information -->
             <left_joint>left_wheel_joint</left_joint>
             <right_joint>right_wheel_joint</right_joint>
-            <!-- kinematics -->
-            <wheel_separation>0.35</wheel_separation>
-            <wheel_diameter>1.0</wheel_diameter>
-            <topic>cmd_vel_joy</topic>
-            <!-- limits -->
+            <wheel_separation>0.297</wheel_separation>
+            <wheel_diameter>0.066</wheel_diameter>
+            <!-- Limits -->
             <max_wheel_torque>200</max_wheel_torque>
             <max_wheel_acceleration>10.0</max_wheel_acceleration>
-            <!-- <min_velocity>0.01</min_velocity>
-            <min_linear_velocity>0.01</min_linear_velocity>
-            <min_angular_velocity>0.01</min_angular_velocity> -->
-            <max_velocity>5.0</max_velocity>
-            <max_linear_velocity>5.0</max_linear_velocity>
-            <max_angular_velocity>6.28</max_angular_velocity>
-            <!-- <min_acceleration>0.01</min_acceleration>
-            <min_linear_acceleration>0.01</min_linear_acceleration>
-            <min_angular_acceleration>0.01</min_angular_acceleration> -->
-            <max_acceleration>5.0</max_acceleration>
-            <max_linear_accelration>5.0</max_linear_accelration>
-            <max_angular_acceleration>6.28</max_angular_acceleration>
-             <!-- publish tf frames -->
-            <odom_topic>odom</odom_topic>
-            <tf_topic>tf</tf_topic>
+            <!-- Output -->
+            <odometry_frame>odom</odometry_frame>
+            <robot_base_frame>base_link</robot_base_frame>
             <publish_odom>true</publish_odom>
             <publish_odom_tf>true</publish_odom_tf>
             <publish_wheel_tf>true</publish_wheel_tf>
-            <frame_id>odom</frame_id>
-            <child_frame_id>base_footprint</child_frame_id>
-            <odom_publish_frequency>50</odom_publish_frequency>
         </plugin>
     </gazebo>

File: src/articubot_one/description/robot_core.xacro (robot description, xacro)
@@ -31,14 +31,14 @@
         <color rgba="1 0 0 1"/>
     </material>
-    <!-- BASE LINK -->
-    <link name="base_footprint">
+     <!-- BASE LINK -->
+    <link name="base_link">
     </link>
     <!-- BASE_FOOTPRINT LINK -->
     <joint name="base_footprint_joint" type="fixed">
-        <parent link="base_footprint"/>
-        <child link="base_link"/>
+        <parent link="base_link"/>
+        <child link="base_footprint"/>
         <origin xyz="0 0 0" rpy="0 0 0"/>
     </joint>
-    <link name="base_link">
+    <link name="base_footprint">
     </link>
     <!-- CHASSIS LINK -->
