Commit message: "Found bug causing issues for nav2, was foxy code leaked into humble in ros2_control and lidar"

File: src/articubot_one/description/lidar.xacro (robot description, xacro)
@@ -30,9 +30,9 @@
     </link>
     <gazebo reference="laser_frame">
-           <material>Gazebo/FlatBlack</material>
-        <sensor type="ray" name="laser">
-            <pose>0 0 0 0 0 0</pose>
-            <visualize>true</visualize>
-            <update_rate>1</update_rate>
+        <material>Gazebo/Black</material>
+        <sensor name="laser" type="ray">
+            <pose> 0 0 0 0 0 0 </pose>
+            <visualize>false</visualize>
+            <update_rate>10</update_rate>
             <ray>
                 <scan>
